File: stm32g474/stm32g474.kicad_pcb (KiCad board)
At the start: 2 copper layers, 57.1 x 38.1 mm, 23 parts, among them U1 STM32G474CBTx, Y1 8Mhz SMD3225-4P, Y2 32.768kHz SMD3215-2P

Commit message: update-2025-11-20
Parts:
- BOOT1: footprint Button_Switch_SMD:SW_SPST_TS-1088-xR020 -> Button_Switch_SMD:SW_SPDT_PCM12
- C3, C4: value 12.5p -> 12p
- moved BOOT1 1.50 mm to (117.8, 50.6)
- turned R2 to 180 degrees
Connections:
- BOOT1 pad 2: BOOT0 -> Net-(BOOT1-B)
- R2 pad 1: GND -> BOOT0
- R2 pad 2: BOOT0 -> Net-(BOOT1-B)
Routing:
- net Net-(BOOT1-B): track 0.00 -> 31.4 mm, vias 0 -> 2
- net BOOT0: track 31.7 -> 7.76 mm, vias 3 -> 0
- net +3V3: track 96.2 -> 91.8 mm, vias 9 -> 8
Other:
- board text added: "OPTIONAL"
