File: stm32g474/stm32g474.kicad_sch (KiCad schematic)
At the start: 23 parts, among them U1 STM32G474CBTx, Y1 8Mhz SMD3225-4P, Y2 32.768kHz SMD3215-2P

Commit message: update-2025-11-20
Parts:
- removed BOOT1: SW-Boot, Button_Switch_SMD:SW_SPST_TS-1088-xR020, symbol atelier-microcontrollers:SW_Push_Small
- added BOOT1: SW-Boot, Button_Switch_SMD:SW_SPDT_PCM12, symbol atelier-microcontrollers:SW_SPDT_123
- C3, C4: value 12.5p -> 12p
Connections:
- net +3V3: now also BOOT1.1 (A)
- net BOOT0: now also R2.1; no longer R2.2
- net GND: now also BOOT1.3 (C); no longer R2.1
- new net: BOOT1.2 (B), R2.2
Other:
- moved on the sheet: C10, R2
